File: Cordillera.kicad_pcb (KiCad board)
At the start: 2 copper layers, 337.2 x 122.6 mm, 208 parts, among them Q1 AO3400, Q2 AO3400, SW1 SW_SPST, U1 STM32F072CBTx, U2 XC6206P332MR, U3 SRV05-4

Commit message: Finish column routing
Parts:
- moved C6 6.03 mm to (156.4, 34.8), turned to 0 degrees
- moved C8 5.29 mm to (148.0, 39.2), turned to 0 degrees
- moved R5 4.53 mm to (147.9, 26.8), turned to 270 degrees
- moved C2 2.84 mm to (148.0, 40.8), turned to 0 degrees
- moved R6 1.26 mm to (150.2, 28.4)
- moved C3 1.19 mm to (156.4, 37.6)
- moved Q1 0.76 mm to (150.5, 25.8)
- moved C4 0.41 mm to (151.1, 54.8)
- moved C1 0.31 mm to (151.1, 53.2)
- moved C5 0.28 mm to (159.9, 49.9)
Connections:
- D10 pad 3: /Switch + LED Matrix/row1 -> /SWDIO
- D11 pad 3: /Switch + LED Matrix/row2 -> /B9
- D14 pad 3: /Switch + LED Matrix/row1 -> /SWDIO
- D15 pad 3: /Switch + LED Matrix/row2 -> /B9
- D19 pad 3: /Switch + LED Matrix/row1 -> /SWDIO
- D2 pad 3: /Switch + LED Matrix/row1 -> /SWDIO
- D20 pad 3: /Switch + LED Matrix/row1 -> /SWDIO
- D21 pad 3: /Switch + LED Matrix/row2 -> /B9
- D24 pad 3: /Switch + LED Matrix/row1 -> /SWDIO
- D25 pad 3: /Switch + LED Matrix/row2 -> /B9
- D29 pad 3: /Switch + LED Matrix/row1 -> /SWDIO
- D3 pad 3: /Switch + LED Matrix/row2 -> /B9
- D30 pad 3: /Switch + LED Matrix/row2 -> /B9
- D33 pad 3: /Switch + LED Matrix/row1 -> /SWDIO
- D34 pad 3: /Switch + LED Matrix/row2 -> /B9
- D5 pad 3: /Switch + LED Matrix/row1 -> /SWDIO
- D6 pad 3: /Switch + LED Matrix/row2 -> /B9
- KBA1 pad 1: /Switch + LED Matrix/colA -> /B15
- KBA2 pad 1: /Switch + LED Matrix/colA -> /B15
- KBA3 pad 1: /Switch + LED Matrix/colA -> /B15
- KBB1 pad 1: /Switch + LED Matrix/colB -> /B14
- KBB2 pad 1: /Switch + LED Matrix/colB -> /B14
- KBB3 pad 1: /Switch + LED Matrix/colB -> /B14
- KBB3-1 pad 1: /Switch + LED Matrix/colB -> /B14
- KBB4 pad 1: /Switch + LED Matrix/colB -> /B14
- KBB5 pad 1: /Switch + LED Matrix/colB -> /B14
- KBC1 pad 1: /Switch + LED Matrix/colC -> /B13
- KBC2 pad 1: /Switch + LED Matrix/colC -> /B13
- KBC3 pad 1: /Switch + LED Matrix/colC -> /B13
- KBC4 pad 1: /Switch + LED Matrix/colC -> /B13
- KBD1 pad 1: /Switch + LED Matrix/colD -> /B12
- KBD2 pad 1: /Switch + LED Matrix/colD -> /B12
- KBD3 pad 1: /Switch + LED Matrix/colD -> /B12
- KBD4 pad 1: /Switch + LED Matrix/colD -> /B12
- KBD5 pad 1: /Switch + LED Matrix/colD -> /B12
- KBE1 pad 1: /Switch + LED Matrix/colE -> /B11
- KBE2 pad 1: /Switch + LED Matrix/colE -> /B11
- KBE3 pad 1: /Switch + LED Matrix/colE -> /B11
- KBE4 pad 1: /Switch + LED Matrix/colE -> /B11
- KBF1 pad 1: /Switch + LED Matrix/colF -> /B10
- KBF2 pad 1: /Switch + LED Matrix/colF -> /B10
- KBF3 pad 1: /Switch + LED Matrix/colF -> /B10
- KBF4 pad 1: /Switch + LED Matrix/colF -> /B10
- KBF5 pad 2: /Switch + LED Matrix/colF -> /B10
- KBF5-1 pad 2: /Switch + LED Matrix/colF -> /B10
- KBG1 pad 1: /Switch + LED Matrix/colG -> /B2
- KBG2 pad 1: /Switch + LED Matrix/colG -> /B2
- KBG3 pad 1: /Switch + LED Matrix/colG -> /B2
- KBG4 pad 1: /Switch + LED Matrix/colG -> /B2
- KBG5 pad 2: /Switch + LED Matrix/colG -> /B2
- KBG5-1 pad 2: /Switch + LED Matrix/colG -> /B2
- KBH1 pad 1: /Switch + LED Matrix/colH -> /A9
- U1 pad 20: Net-(U1-Pad20) -> /B2
- U1 pad 21: Net-(U1-Pad21) -> /B10
- U1 pad 22: Net-(U1-Pad22) -> /B11
- U1 pad 25: Net-(U1-Pad25) -> /B12
- U1 pad 26: Net-(U1-Pad26) -> /B13
- U1 pad 27: Net-(U1-Pad27) -> /B14
- U1 pad 28: Net-(U1-Pad28) -> /B15
- U1 pad 30: Net-(U1-Pad30) -> /A9
- U1 pad 46: Net-(U1-Pad46) -> /B9
Routing:
- net /B14: track 0.00 -> 229.3 mm
- net /SWDIO: track 0.00 -> 216.2 mm, vias 0 -> 2
- net /B15: track 0.00 -> 210.4 mm
- net /Switch + LED Matrix/colB: track 206.0 -> 0.00 mm
- net /B9: track 0.00 -> 192.0 mm
- net /Switch + LED Matrix/colA: track 186.6 -> 0.00 mm
- net /B12: track 0.00 -> 182.0 mm
- net /B13: track 0.00 -> 177.1 mm
- net /Switch + LED Matrix/row1: track 164.2 -> 0.00 mm
- net /Switch + LED Matrix/colD: track 159.8 -> 0.00 mm
- net /Switch + LED Matrix/colC: track 154.4 -> 0.00 mm
- net /B10: track 0.00 -> 143.4 mm
- net /B11: track 0.00 -> 142.1 mm
- net /B2: track 0.00 -> 133.9 mm
- net /Switch + LED Matrix/row2: track 133.3 -> 0.00 mm
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
Commit message: Update files
Parts:
- added J1: Conn_01x08, keeb_connectors:PinHeader_2x04_P2.54mm_Vertical, B.Cu at (142.4, 32.2)
- C1, C10, C2, C3, C4, C5, C6, C7, C8, C9: footprint keeb_parts:R_0603_1608Metric -> keeb_parts:C_0603_1608Metric
- C11: value 1u -> 4.7u; footprint keeb_parts:R_0603_1608Metric -> keeb_parts:C_0603_1608Metric
- C12: value 470n -> 1u; footprint keeb_parts:R_0603_1608Metric -> keeb_parts:C_0603_1608Metric
- Q1, Q2: value AO3400 -> 2N7002
- moved R7 27.3 mm to (164.8, 53.5), turned to 0 degrees
- moved R4 23.4 mm to (164.8, 50.0), turned to 180 degrees
- moved C11 21.9 mm to (164.8, 51.8), turned to 180 degrees
- moved Q2 21.7 mm to (164.8, 56.3), turned to 270 degrees
- moved C12 20.1 mm to (151.0, 56.6), turned to 180 degrees
- moved R77 14.3 mm to (-3.74, 71.4), turned to 90 degrees
- moved SW1 13.2 mm to (157.4, 57.1), turned to 0 degrees
- moved R76 10.2 mm to (-5.34, 71.4), turned to 90 degrees
- moved R8 9.45 mm to (151.0, 58.3), turned to 180 degrees
- moved R75 7.04 mm to (-6.94, 71.4), turned to 90 degrees
- moved D1 3.80 mm to (151.4, -2.49)
- moved U3 3.41 mm to (159.4, -2.49)
- moved F1 3.10 mm to (154.6, -2.49)
- moved U2 2.98 mm to (154.6, 3.30)
- moved C10 2.85 mm to (154.5, 6.01)
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Connections:
- net Net-(U1-Pad2) renamed /C13
- net Net-(U1-Pad3) renamed /C14
- net Net-(U1-Pad4) renamed /C15
- net Net-(U1-Pad5) renamed /F0
- D12 pad 3: /Switch + LED Matrix/row3 -> /F1
- D13 pad 3: /Switch + LED Matrix/row4 -> /A10
- D16 pad 3: /Switch + LED Matrix/row3 -> /F1
- D17 pad 3: /Switch + LED Matrix/row4 -> /A10
- D18 pad 3: /Switch + LED Matrix/row5 -> /A9
- D22 pad 3: /Switch + LED Matrix/row3 -> /F1
- D23 pad 3: /Switch + LED Matrix/row4 -> /A10
- D26 pad 3: /Switch + LED Matrix/row3 -> /F1
- D27 pad 3: /Switch + LED Matrix/row4 -> /A10
- D28 pad 3: /Switch + LED Matrix/row5 -> /A9
- D31 pad 3: /Switch + LED Matrix/row3 -> /F1
- D32 pad 3: /Switch + LED Matrix/row4 -> /A10
- D35 pad 3: /Switch + LED Matrix/row3 -> /F1
- D36 pad 3: /Switch + LED Matrix/row4 -> /A10
- D37 pad 3: /Switch + LED Matrix/row5 -> /A9
- D4 pad 3: /Switch + LED Matrix/row3 -> /F1
- D7 pad 3: /Switch + LED Matrix/row3 -> /F1
- D8 pad 3: /Switch + LED Matrix/row4 -> /A10
- D9 pad 3: /Switch + LED Matrix/row5 -> /A9
- KBH1 pad 1: /A9 -> /B1
- R75 pad 2: /LED_1 -> /B0
- R76 pad 2: /LED_2 -> /A1
- R77 pad 2: /LED_3 -> /A0
- R8 pad 1: +3V3 -> /NRST
- R8 pad 2: /NRST -> +3V3
- U1 pad 10: Net-(U1-Pad10) -> /A0
- U1 pad 11: Net-(U1-Pad11) -> /A1
- U1 pad 18: Net-(U1-Pad18) -> /B0
- U1 pad 19: Net-(U1-Pad19) -> /B1
- U1 pad 31: Net-(U1-Pad31) -> /A10
- U1 pad 6: Net-(U1-Pad6) -> /F1
- U3 pad 1: Net-(U3-Pad1) -> /D+
- U3 pad 3: Net-(U3-Pad3) -> /D+
- U3 pad 4: Net-(U3-Pad4) -> /D-
- U3 pad 6: Net-(U3-Pad6) -> /D-
Routing:
- net GND: track 52.4 -> 401.0 mm, vias 3 -> 11
- net /A9: track 41.7 -> 301.7 mm, vias 0 -> 2
- net /A10: track 0.00 -> 239.4 mm, vias 0 -> 2
- net /Switch + LED Matrix/row5: track 238.6 -> 0.00 mm
- net /A0: track 0.00 -> 207.5 mm, vias 0 -> 2
- net /F1: track 0.00 -> 205.7 mm, vias 0 -> 4
- net /B0: track 0.00 -> 202.4 mm, vias 0 -> 2
- net /A1: track 0.00 -> 195.3 mm, vias 0 -> 2
- net /Switch + LED Matrix/row3: track 186.6 -> 0.00 mm
- net /Switch + LED Matrix/row4: track 174.4 -> 0.00 mm
- net +3V3: track 81.5 -> 143.0 mm, vias 4 -> 6
- net /B1: track 0.00 -> 39.0 mm, vias 0 -> 1
- net +5V: track 1818.2 -> 1853.4 mm, vias 0 -> 3
- net /NRST: track 0.00 -> 26.0 mm, vias 0 -> 2
- net /SPI_SCK: track 0.00 -> 24.3 mm, vias 0 -> 1
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Other:
- outline, holes or cut-outs redrawn
- board text added: "+3V3"
- board text added: "CS"
- board text added: "GND"
- board text added: "IRQ"
- board text added: "MISO"
- board text added: "MOSI"
- board text added: "RES"
- board text added: "SCK"
